File: V5/Hw/Magspoof_V5.kicad_pcb (KiCad board)
At the start: 2 copper layers, 76.5 x 32.5 mm, 59 parts, among them J1 SWD, J2 SWD, P1 USB_C_Plug_USB2.0, Q1 DMG3415U-7, SW1 ON, SW3 S1, SW4 SOURCE MAG, SW5 RESET, U1 CH552G, U2 AP2112K-3.3, U3 TC4424, U5 MCP73831

Commit message: feat(hw): BOM got updated
Routing:
- net /D-: track 20.7 -> 23.9 mm
- net GND: vias 32 -> 36
Changed lines of the file:
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@@
+	)
+	(via
+		(at 105.5 42.25)
+		(size 0.6)
+		(drill 0.3)
+		(layers "F.Cu" "B.Cu")
+		(free yes)
+		(net 2)
 	)
 	(via
@@
 	)
 	(via
+		(at 104.75 41.5)
+		(size 0.6)
+		(drill 0.3)
+		(layers "F.Cu" "B.Cu")
+		(free yes)
+		(net 2)
+	)
+	(via
 		(at 110.5 47.55)
 		(size 0.6)
@@
 	(via
 		(at 122 42)
+		(size 0.6)
+		(drill 0.3)
+		(layers "F.Cu" "B.Cu")
+		(free yes)
+		(net 2)
+	)
+	(via
+		(at 104.75 42.25)
+		(size 0.6)
+		(drill 0.3)
+		(layers "F.Cu" "B.Cu")
+		(free yes)
+		(net 2)
+	)
+	(via
+		(at 105.5 41.5)
 		(size 0.6)
 		(drill 0.3)
@@
 	)
 	(segment
+		(start 107 50.015)
+		(end 106.75 50.015)
+		(width 0.2)
+		(layer "F.Cu")
+		(net 15)
+	)
+	(segment
+		(start 106.75 49.765)
+		(end 107 50.015)
+		(width 0.2)
+		(layer "F.Cu")
+		(net 15)
+	)
+	(segment
 		(start 122.235 47.690001)
 		(end 122.645 48.100001)
@@
 	)
 	(segment
+		(start 106.75 49.25)
+		(end 106.49 48.99)
+		(width 0.2)
+		(layer "F.Cu")
+		(net 15)
+	)
+	(segment
+		(start 106.75 49.75)
+		(end 106.75 49.765)
+		(width 0.2)
+		(layer "F.Cu")
+		(net 15)
+	)
+	(segment
+		(start 106.75 50.015)
+		(end 106.5 50.015)
+		(width 0.2)
+		(layer "F.Cu")
+		(net 15)
+	)
+	(segment
+		(start 121.9468 50.015)
+		(end 107 50.015)
+		(width 0.2)
+		(layer "F.Cu")
+		(net 15)
+	)
+	(segment
 		(start 122.645 49.3168)
 		(end 121.9468 50.015)
@@
 	)
 	(segment
-		(start 121.9468 50.015)
+		(start 106.49 48.99)
+		(end 105.205 48.99)
+		(width 0.2)
+		(layer "F.Cu")
+		(net 15)
+	)
+	(segment
+		(start 106.75 50.015)
+		(end 106.75 49.75)
+		(width 0.2)
+		(layer "F.Cu")
+		(net 15)
+	)
+	(segment
+		(start 106.5 50.015)
 		(end 106.467501 50.015)
 		(width 0.2)
@@
 	)
 	(segment
+		(start 106.75 49.75)
+		(end 106.75 49.25)
+		(width 0.2)
+		(layer "F.Cu")
+		(net 15)
+	)
+	(segment
 		(start 106.467501 50.015)
 		(end 106.442501 49.99)
 		(width 0.2)
 		(layer "F.Cu")
+		(net 15)
+	)
+	(segment
+		(start 106.75 49.765)
+		(end 106.5 50.015)
+		(width 0.2)
+		(layer "F.Cu")
